Commit message: done

File: body.urdf (robot description, URDF)
Before this commit: robot robot, 9 links, 8 joints
Links:
- removed link LinkBackLeg
- removed link LinkFrontLeg
- removed link LinkLeftLeg
- removed link LinkLowerBackLeg
- removed link LinkLowerFrontLeg
- removed link LinkLowerLeftLeg
- removed link LinkLowerRightLeg
- removed link LinkRightLeg
- removed link LinkTorso
- added link Link1, mass 1; collision box size=1 0.5 0.5; visual box size=1 0.5 0.5
- added link Link2, mass 1; collision box size=1 0.5 0.5; visual box size=1 0.5 0.5
- added link Link3, mass 1; collision box size=1 0.5 0.5; visual box size=1 0.5 0.5
- added link Link4, mass 1; collision box size=1 0.5 0.5; visual box size=1 0.5 0.5
Joints:
- removed joint LinkBackLeg_LinkLowerBackLeg
- removed joint LinkFrontLeg_LinkLowerFrontLeg
- removed joint LinkLeftLeg_LinkLowerLeftLeg
- removed joint LinkRightLeg_LinkLowerRightLeg
- removed joint LinkTorso_LinkBackLeg
- removed joint LinkTorso_LinkFrontLeg
- removed joint LinkTorso_LinkLeftLeg
- removed joint LinkTorso_LinkRightLeg
- added joint Link1_Link2: type revolute, parent Link1, child Link2, origin xyz=0.5 0 1.5 rpy=0 0 0, axis 0 1 0, limit lower=-3.14159 upper=3.14159 effort=0.0 velocity=0.0
- added joint Link2_Link3: type revolute, parent Link2, child Link3, origin xyz=1 0 0 rpy=0 0 0, axis 0 1 0, limit lower=-3.14159 upper=3.14159 effort=0.0 velocity=0.0
- added joint Link3_Link4: type revolute, parent Link3, child Link4, origin xyz=1 0 0 rpy=0 0 0, axis 0 0 1, limit lower=-3.14159 upper=3.14159 effort=0.0 velocity=0.0
